File: Pure Noise.brd (EAGLE design)
At the start: 18.3 x 100 mm, 45 parts

Commit message: Noise 1.1
Parts:
- removed R16, R17: 100K, rcl:R0805
- C9: value 0.1u -> 0.22uF***
- R11: value 9K1*** -> 39K***
- R12: value 100K -> 5K6***
- R13: value 560K -> 100K
Connections:
- removed net N$7: R16.1, R17.1, U$6.3-IN
- net GND: no longer R17.2
- net PINK: now also U$6.3-IN; no longer R16.2
Routing:
- net N$7: track 5.61 -> 0.00 mm
- net PINK: track 39.2 -> 43.3 mm
Other:
- board text added: "Pure Nz V1.1"
- board text added: "copywrite GMSN Ltd 2016"
- board text removed: "Designed by Jason H. J. Lim and Rob Spencer copyright GMSN Ltd 2016"
- board text removed: "Pure Nz V1.0"

Commit message: Reinstall
Parts:
- removed C14, C15: 0.1u, rcl:C0805K
- removed U$1: DUAL_OPAMP, INSTRUO:DUAL_OPAMP
- removed U$2: (no value), gmsnLogo:GMSN!_LOGO
- removed U$6: QUAD_OPAMP, QuBit:QUAD_OPAMP
- removed U$9: TRANS_PAIR, QuBit:TRANS_PAIR
- added IC3: OPAMP_DUALD, GMSN:SO08
- added IC4: OPAMP_QUADD, GMSN:SO14
- added T1: TRANSISTOR_PAIR_NPN, GMSN:TRANS_PAIR
- BLUE, PINK, RED, WHITE: value (none) -> SOCKET_MONO_3.5MMPJ301M-12; device INSTRUO:S_JACK -> GMSN:PJ301M-12
- C1, C2: device rcl:153CLV-0505 -> GMSN:153CLV-0505
- C10, C11, C12, C13, C4, C5, C6, C7, C8, C9: device rcl:C0805K -> GMSN:C0805
- C3: device rcl:C1206K -> GMSN:C0805
- D1, D2: device adafruit:SMADIODE -> GMSN:SMADIODE
- JP1: value M05X2SHD -> HEADER2X5SHD; device SparkFun-Connectors:2X5-SHROUDED -> GMSN:2X5-SHROUDED
- R1, R10, R11, R12, R13, R14, R15, R2, R3, R4, R5, R6, R7, R8, R9: device rcl:R0805 -> GMSN:R0805
- TR1: device INSTRUO:TRIM_3269W -> GMSN:TRIMMER_TH
- moved C11 51.7 mm to (3.81, 94.8)
- moved C10 38.6 mm to (16.0, 89.3)
- moved R1 34.2 mm to (6.19, 77.2), turned to 180 degrees
- moved R15 33.4 mm to (6.19, 97.3)
- moved R2 32.1 mm to (6.19, 57.1), turned to 180 degrees
- moved R5 24.8 mm to (3.81, 92.8)
- moved R11 22.0 mm to (3.81, 86.6), turned to 180 degrees
- moved R13 21.3 mm to (16.0, 87.1), turned to 180 degrees
- moved R14 20.7 mm to (6.19, 43.3), turned to 180 degrees
- moved R4 19.9 mm to (3.89, 84.5), turned to 180 degrees
- moved R8 19.7 mm to (7.62, 69.8)
- moved C9 18.9 mm to (16.0, 84.8), turned to 180 degrees
- moved R7 18.7 mm to (9.84, 66.0), turned to 180 degrees
- moved U$3 17.8 mm to (9.92, 112.1), flipped to the bottom
- moved C7 15.5 mm to (5.24, 69.8), turned to 90 degrees
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Connections:
- removed net N$8: R14.1, U$6.1OUT
- new net N$7: C9.2, IC4.1, R13.2, R14.1
- net +12V: now also IC3.8, IC4.4; no longer C14.1, U$1.+VCC, U$6.VCC++
- net -12V: now also IC3.4, IC4.11; no longer C15.2, U$1.-VCC, U$6.VCC--
- net BLUE: no longer R11.1
- net GND: now also IC3.3, IC4.3, IC4.5, T1.4; no longer C14.2, C15.1, U$1.+1IN, U$6.1+IN, U$6.2+IN, U$9.E1
- net N$1: now also IC3.6, IC3.7; no longer U$1.2OUT
- net N$11: now also IC4.14, R11.1; no longer U$6.4OUT
- net N$12: now also T1.1, T1.2; no longer U$9.B1, U$9.B2
- net N$13: now also T1.5; no longer U$9.E2
- net N$14: now also T1.3; no longer U$9.C1
- net N$15: now also IC3.2; no longer U$1.-1IN
- net N$16: now also IC4.6; no longer U$6.2-IN
- net N$19: now also IC3.1, IC3.5; no longer U$1.+2IN, U$1.1OUT
- net N$2: now also IC4.8, IC4.9; no longer U$6.3OUT
- net N$23: now also IC4.10, IC4.7; no longer U$6.2OUT, U$6.3+IN
- net N$4: now also IC4.13; no longer U$6.4+IN
- net N$5: now also IC4.12; no longer U$6.4-IN
- net N$6: now also IC4.2; no longer U$6.1-IN
- net PINK: no longer U$6.3-IN
- net RED: no longer C9.2, R13.2
- net WHITE: no longer U$1.-2IN
Routing:
- net N$7: track 0.00 -> 59.0 mm, vias 0 -> 2
- net WHITE: track 48.2 -> 3.13 mm, vias 3 -> 0
- net BLUE: track 47.5 -> 2.97 mm, vias 1 -> 0
- net N$19: track 57.2 -> 14.5 mm, vias 4 -> 0
- net PINK: track 43.3 -> 3.21 mm, vias 2 -> 0
- net RED: track 40.2 -> 3.12 mm
- net -12V: track 63.6 -> 100.5 mm
- net N$2: track 17.3 -> 49.9 mm, vias 0 -> 2
- net +12V: track 75.7 -> 101.2 mm, vias 4 -> 0
- net N$11: track 3.66 -> 14.5 mm, vias 0 -> 2
- net N$15: track 7.82 -> 17.7 mm
- net N$5: track 8.54 -> 14.6 mm, vias 0 -> 3
- net N$1: track 6.55 -> 11.4 mm
- net N$6: track 13.9 -> 9.25 mm
- net N$8: track 3.67 -> 0.00 mm
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Other:
- board text added: "Pure Noise v1.2 cc-by 4.0 2021 The Little Red Hen"
- board text removed: "Pure Nz V1.1"
- board text removed: "copywrite GMSN Ltd 2016"
- board text removed: "power"
