File: Pure Noise.sch (EAGLE design)
At the start: 43 parts

Commit message: Noise 1.1
Parts:
- removed R16, R17: 100K, rcl:R-US_R0805
- C9: value 0.1u -> 0.22uF***
- R11: value 9K1*** -> 39K***
- R12: value 100K -> 5K6***
- R13: value 560K -> 100K
Connections:
- removed net N$7: R16.1, R17.1, U$6G$3.-IN
- net GND: no longer R17.2
- net PINK: now also U$6G$3.-IN; no longer R16.2
Other:
- note added: "5K6***"
Changed lines of the file:
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@@
 <?xml version="1.0" encoding="utf-8"?>
 <!DOCTYPE eagle SYSTEM "eagle.dtd">
-<eagle version="7.2.0">
+<eagle version="7.1.0">
 <drawing>
 <settings>
@@
 <part name="GND2" library="supply1" deviceset="GND" device=""/>
 <part name="R5" library="rcl" deviceset="R-US_" device="R0805" value="200K"/>
-<part name="R11" library="rcl" deviceset="R-US_" device="R0805" value="9K1***"/>
-<part name="R12" library="rcl" deviceset="R-US_" device="R0805" value="100K"/>
-<part name="R13" library="rcl" deviceset="R-US_" device="R0805" value="560K"/>
-<part name="C9" library="rcl" deviceset="C-US" device="C0805K" value="0.1u"/>
+<part name="R11" library="rcl" deviceset="R-US_" device="R0805" value="39K***"/>
+<part name="R12" library="rcl" deviceset="R-US_" device="R0805" value="5K6***"/>
+<part name="R13" library="rcl" deviceset="R-US_" device="R0805" value="100K"/>
+<part name="C9" library="rcl" deviceset="C-US" device="C0805K" value="0.22uF***"/>
 <part name="R14" library="rcl" deviceset="R-US_" device="R0805" value="1K"/>
 <part name="GND3" library="supply1" deviceset="GND" device=""/>
@@
 <part name="C14" library="rcl" deviceset="C-US" device="C0805K" value="0.1u"/>
 <part name="C15" library="rcl" deviceset="C-US" device="C0805K" value="0.1u"/>
-<part name="R16" library="rcl" deviceset="R-US_" device="R0805" value="100K"/>
-<part name="R17" library="rcl" deviceset="R-US_" device="R0805" value="100K"/>
-<part name="GND6" library="supply1" deviceset="GND" device=""/>
 </parts>
 <sheets>
@@
 <plain>
 <text x="160.02" y="111.76" size="1.778" layer="91">22K</text>
+<text x="210.82" y="119.38" size="1.778" layer="91">5K6***</text>
 </plain>
 <instances>
@@
 <instance part="C14" gate="G$1" x="152.4" y="35.56"/>
 <instance part="C15" gate="G$1" x="152.4" y="22.86"/>
-<instance part="R16" gate="G$1" x="228.6" y="81.28"/>
-<instance part="R17" gate="G$1" x="228.6" y="96.52"/>
-<instance part="GND6" gate="1" x="238.76" y="91.44"/>
 </instances>
 <busses>
@@
 <pinref part="GND5" gate="1" pin="GND"/>
 </segment>
-<segment>
-<pinref part="R17" gate="G$1" pin="2"/>
-<wire x1="233.68" y1="96.52" x2="238.76" y2="96.52" width="0.1524" layer="91"/>
-<wire x1="238.76" y1="96.52" x2="238.76" y2="93.98" width="0.1524" layer="91"/>
-<pinref part="GND6" gate="1" pin="GND"/>
-</segment>
 </net>
 <net name="+12V" class="0">
@@
 <wire x1="251.46" y1="68.58" x2="248.92" y2="68.58" width="0.1524" layer="91"/>
 <junction x="251.46" y="68.58"/>
-<pinref part="R16" gate="G$1" pin="2"/>
-<wire x1="233.68" y1="81.28" x2="251.46" y2="81.28" width="0.1524" layer="91"/>
+<pinref part="U$6" gate="G$3" pin="-IN"/>
+<wire x1="210.82" y1="73.66" x2="208.28" y2="73.66" width="0.1524" layer="91"/>
+<wire x1="208.28" y1="73.66" x2="208.28" y2="81.28" width="0.1524" layer="91"/>
+<wire x1="251.46" y1="81.28" x2="208.28" y2="81.28" width="0.1524" layer="91"/>
 </segment>
 <segment>
@@
 </segment>
 </net>
-<net name="N$7" class="0">
-<segment>
-<pinref part="U$6" gate="G$3" pin="-IN"/>
-<wire x1="210.82" y1="73.66" x2="208.28" y2="73.66" width="0.1524" layer="91"/>
-<wire x1="208.28" y1="73.66" x2="208.28" y2="81.28" width="0.1524" layer="91"/>
-<pinref part="R16" gate="G$1" pin="1"/>
-<wire x1="223.52" y1="81.28" x2="218.44" y2="81.28" width="0.1524" layer="91"/>
-<pinref part="R17" gate="G$1" pin="1"/>
-<wire x1="218.44" y1="81.28" x2="208.28" y2="81.28" width="0.1524" layer="91"/>
-<wire x1="223.52" y1="96.52" x2="218.44" y2="96.52" width="0.1524" layer="91"/>
-<wire x1="218.44" y1="96.52" x2="218.44" y2="81.28" width="0.1524" layer="91"/>
-<junction x="218.44" y="81.28"/>
-</segment>
-</net>

Commit message: Reinstall
Parts:
- removed C14, C15: 0.1u, rcl:C-USC0805K
- removed U$1: DUAL_OPAMP, INSTRUO:DUAL_OPAMP
- removed U$6: QUAD_OPAMP, QuBit:QUAD_OPAMP
- removed U$9: TRANS_PAIR, QuBit:TRANS_PAIR
- added IC3: OPAMP_DUALD, GMSN:OPAMP_DUALD
- added IC4: OPAMP_QUADD, GMSN:OPAMP_QUADD
- added T1: TRANSISTOR_PAIR_NPN, GMSN:TRANSISTOR_PAIR_NPN
- BLUE, PINK, RED, WHITE: value S_JACK -> SOCKET_MONO_3.5MMPJ301M-12; device INSTRUO:S_JACK -> GMSN:SOCKET_MONO_3.5MMPJ301M-12
- C1, C2: device rcl:CPOL-US153CLV-0505 -> GMSN:CAPACITOR_POL-US153CLV-0505
- C10, C11, C12, C13, C4, C5, C6, C7, C8, C9: device rcl:C-USC0805K -> GMSN:CAPACITOR-USC0805
- C3: device rcl:C-USC1206K -> GMSN:CAPACITOR-USC0805
- D1, D2: device adafruit:DIODESMA -> GMSN:DIODESMA
- JP1: value M05X2SHD -> HEADER2X5SHD; device SparkFun-Connectors:M05X2SHD -> GMSN:HEADER2X5SHD
- R1, R10, R11, R12, R13, R14, R15, R2, R3, R4, R5, R6, R7, R8, R9: device rcl:R-US_R0805 -> GMSN:RESISTOR_USR0805
- TR1: device INSTRUO:TRIM_3269W -> GMSN:RESISTOR_VARIABLETRIMMER_TH
Connections:
- removed net N$8: R14.1, U$6G$1.OUT
- new net N$7: C9.2, IC4A.OUT, R13.2, R14.1
- net +12V: now also IC3P.V+, IC4P.V+; no longer C14.1, U$1G$3.+12V, U$6G$5.+12V
- net -12V: now also IC3P.V-, IC4P.V-; no longer C15.2, U$1G$4.-12V, U$6G$6.-12V
- net BLUE: no longer R11.1
- net GND: now also BLUE.SLEEVE, IC3A.+IN, IC4A.+IN, IC4B.+IN, PINK.SLEEVE, RED.SLEEVE, T1G$1.E, WHITE.SLEEVE; no longer BLUE.GND, C14.2, C15.1, PINK.GND, RED.GND, U$1G$1.+IN, U$6G$1.+IN, U$6G$2.+IN, U$9G$1.E, WHITE.GND
- net N$1: now also IC3B.-IN, IC3B.OUT; no longer U$1G$2.OUT
- net N$11: now also IC4D.OUT, R11.1; no longer U$6G$4.OUT
- net N$12: now also T1G$1.B, T1G$2.B; no longer U$9G$1.B, U$9G$2.B
- net N$13: now also T1G$2.E; no longer U$9G$2.E
- net N$14: now also T1G$1.C; no longer U$9G$1.C
- net N$15: now also IC3A.-IN; no longer U$1G$1.-IN
- net N$16: now also IC4B.-IN; no longer U$6G$2.-IN
- net N$19: now also IC3A.OUT, IC3B.+IN; no longer U$1G$1.OUT, U$1G$2.+IN
- net N$2: now also IC4C.-IN, IC4C.OUT; no longer U$6G$3.OUT
- net N$23: now also IC4B.OUT, IC4C.+IN; no longer U$6G$2.OUT, U$6G$3.+IN
- net N$4: now also IC4D.-IN; no longer U$6G$4.+IN
- net N$5: now also IC4D.+IN; no longer U$6G$4.-IN
- net N$6: now also IC4A.-IN; no longer U$6G$1.-IN
- net PINK: no longer U$6G$3.-IN
- net RED: no longer C9.2, R13.2
- net WHITE: no longer U$1G$2.-IN
Other:
- moved on the sheet: R1, R15
